File: hardware/C5VRX_JACK_DIY_V2/C5VRX_JACK_DIY_V2.kicad_pcb (KiCad board)
At the start: 2 copper layers, 42.5 x 28.8 mm, 18 parts, among them J1 FATSHARK BAY, J2 PJ-320D, U1 XIAO ESP32-C5

Commit message: Update REV B README and replace ground bridge with copper pour
Routing:
- net /GND: track 19.2 -> 7.50 mm
- added copper zone on F.Cu, net /GND
Changed lines of the file:
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@@
-	)
-	(segment
-		(start 122 124.5)
-		(end 123.5 123)
-		(width 0.4)
-		(layer "F.Cu")
-		(net "/GND")
-	)
-	(segment
-		(start 113.425 126.55)
-		(end 114.5 125.475)
-		(width 0.4)
-		(layer "F.Cu")
-		(net "/GND")
 	)
 	(segment
@@
 	)
 	(segment
-		(start 115.2 124.5)
-		(end 122 124.5)
-		(width 0.4)
-		(layer "F.Cu")
-		(net "/GND")
-	)
-	(segment
 		(start 113.425 126.55)
 		(end 109.85 126.55)
-		(width 0.4)
-		(layer "F.Cu")
-		(net "/GND")
-	)
-	(segment
-		(start 114.5 125.475)
-		(end 114.5 125.2)
-		(width 0.4)
-		(layer "F.Cu")
-		(net "/GND")
-	)
-	(segment
-		(start 114.5 125.2)
-		(end 115.2 124.5)
 		(width 0.4)
 		(layer "F.Cu")
@@
 	)
 	(zone
+		(net "/GND")
+		(layer "F.Cu")
+		(name "GND front")
+		(hatch edge 0.5)
+		(connect_pads
+			(clearance 0.2)
+		)
+		(min_thickness 0.25)
+		(fill yes
+			(thermal_gap 0.25)
+			(thermal_bridge_width 0.3)
+			(island_removal_mode 0)
+		)
+		(polygon
+			(pts
+				(xy 100.4 100.4) (xy 142.11 100.4) (xy 142.11 128.4) (xy 100.4 128.4)
+			)
+		)
+	)
+	(zone
