File: hardware/C5VRX_JACK_DIY_V2/C5VRX_JACK_DIY_V2.kicad_pcb (KiCad board)
At the start: 2 copper layers, 42.5 x 28.8 mm, 18 parts, among them J1 FATSHARK BAY, J2 PJ-320D, U1 XIAO ESP32-C5

Commit message: REV B: R8 15k (D10) and R9 33k (D3) for the 8-bit DAC
- Schematic, PCB (silkscreen value text) and BOM: R8 16k -> 15k,
  R9 32k -> 33k; R1-R7 and the 200 ohm load unchanged
- Regenerate Gerbers, drills, gerber ZIP, schematic/fit-check PDFs,
  SVGs, DRC/ERC reports, the 3D top image and the three front renders
  with KiCad 10.0.7 using the previous export settings; copper, mask
  and drill data are unchanged apart from headers. STEP/GLB and back
  renders carry no resistor values and stay as they were
- Update README, hardware README, AGENTS.md and FINDINGS.md values

Co-Authored-By: Claude Opus 5.5 <noreply@anthropic.com>
Claude-Session: https://claude.ai/code/session_017AWz9uZd39iY6CDkhsBZb6
Parts:
- R8: value 16k -> 15k
- R9: value 32k -> 33k
Changed lines of the file:
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@@
 			)
 		)
-		(property "Value" "32k"
+		(property "Value" "33k"
 			(at 6.98 0 0)
 			(layer "F.SilkS")
@@
 			)
 		)
-		(property "Value" "16k"
+		(property "Value" "15k"
 			(at 6.98 0 0)
 			(layer "F.SilkS")
