File: hardware/C5VRX_JACK_DIY_V2/C5VRX_JACK_DIY_V2.kicad_sch (KiCad schematic)
At the start: 16 parts, among them J1 FATSHARK BAY, J2 PJ-320D, U1 XIAO ESP32-C5

Commit message: REV B: R8 15k (D10) and R9 33k (D3) for the 8-bit DAC
- Schematic, PCB (silkscreen value text) and BOM: R8 16k -> 15k,
  R9 32k -> 33k; R1-R7 and the 200 ohm load unchanged
- Regenerate Gerbers, drills, gerber ZIP, schematic/fit-check PDFs,
  SVGs, DRC/ERC reports, the 3D top image and the three front renders
  with KiCad 10.0.7 using the previous export settings; copper, mask
  and drill data are unchanged apart from headers. STEP/GLB and back
  renders carry no resistor values and stay as they were
- Update README, hardware README, AGENTS.md and FINDINGS.md values

Co-Authored-By: Claude Opus 5.5 <noreply@anthropic.com>
Claude-Session: https://claude.ai/code/session_017AWz9uZd39iY6CDkhsBZb6
Parts:
- R8: value 16k -> 15k
- R9: value 32k -> 33k
Other:
- note added: "REV B: R8 15k / D10 and R9 33k / D3 are DNP. PR259 remains 6-bit. 8-bit: D9..D4 = bits 7..2, D10 = bit 1, D3 = bit 0. Populate only with wider DAC firmware and loaded CVBS / D3 boot validation."
- note removed: "REV B: R8 16k / D10 and R9 32k / D3 are DNP. PR259 remains 6-bit. 8-bit: D9..D4 = bits 7..2, D10 = bit 1, D3 = bit 0. Populate only with wider DAC firmware and loaded CVBS / D3 boot validation."
Changed lines of the file:
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@@
 (symbol (lib_id "C5VRX:R") (at 110.49 55.88 0) (unit 1) (in_bom yes) (on_board yes) (dnp yes)
        (property "Reference" "R8" (at 107.95 53.34 0) (effects (font (size 1.0 1.0))))
-       (property "Value" "16k" (at 114.3 53.34 0) (effects (font (size 1.0 1.0))))
+       (property "Value" "15k" (at 114.3 53.34 0) (effects (font (size 1.0 1.0))))
        (property "Footprint" "Resistor_THT:R_Axial_DIN0207_L6.3mm_D2.5mm_P10.16mm_Horizontal" (at 110.49 55.88 0) (effects (font (size 1 1)) (hide yes)))
        (instances (project "C5VRX_JACK_DIY_V2" (path "/3f7e44b9-0d23-4154-a2e9-c50963f7f4c3" (reference "R8") (unit 1)))))
@@
 (symbol (lib_id "C5VRX:R") (at 110.49 63.5 0) (unit 1) (in_bom yes) (on_board yes) (dnp yes)
        (property "Reference" "R9" (at 107.95 60.96 0) (effects (font (size 1.0 1.0))))
-       (property "Value" "32k" (at 114.3 60.96 0) (effects (font (size 1.0 1.0))))
+       (property "Value" "33k" (at 114.3 60.96 0) (effects (font (size 1.0 1.0))))
        (property "Footprint" "Resistor_THT:R_Axial_DIN0207_L6.3mm_D2.5mm_P10.16mm_Horizontal" (at 110.49 63.5 0) (effects (font (size 1 1)) (hide yes)))
        (instances (project "C5VRX_JACK_DIY_V2" (path "/3f7e44b9-0d23-4154-a2e9-c50963f7f4c3" (reference "R9") (unit 1)))))
@@
     (label "DAC_EXT8" (at 154.94 63.5 0) (effects (font (size 1 1))))
 (label "DAC_EXT8_SW" (at 165.1 63.5 0) (effects (font (size 1 1))))
-(text "REV B: R8 16k / D10 and R9 32k / D3 are DNP.\nPR259 remains 6-bit. 8-bit: D9..D4 = bits 7..2, D10 = bit 1, D3 = bit 0.\nPopulate only with wider DAC firmware and loaded CVBS / D3 boot validation." (at 144.78 45.72 0) (effects (font (size 1 1)) (justify left top)))(text "SJ2 / SJ3: rear, normally OPEN.\n6-bit: both open. 7-bit: close SJ2 only.\n8-bit: close SJ2 + SJ3.\nFit R8/R9 and use matching DAC firmware." (at 144.78 76.2 0) (effects (font (size 1 1)) (justify left top)))
+(text "REV B: R8 15k / D10 and R9 33k / D3 are DNP.\nPR259 remains 6-bit. 8-bit: D9..D4 = bits 7..2, D10 = bit 1, D3 = bit 0.\nPopulate only with wider DAC firmware and loaded CVBS / D3 boot validation." (at 144.78 45.72 0) (effects (font (size 1 1)) (justify left top)))(text "SJ2 / SJ3: rear, normally OPEN.\n6-bit: both open. 7-bit: close SJ2 only.\n8-bit: close SJ2 + SJ3.\nFit R8/R9 and use matching DAC firmware." (at 144.78 76.2 0) (effects (font (size 1 1)) (justify left top)))
 )
