File: hardware/C5VRX_JACK_DIY_V3/C5VRX_JACK_DIY_V3.kicad_pcb (KiCad board)
At the start: 2 copper layers, 42.5 x 28.8 mm, 18 parts, among them J1 FATSHARK BAY, J2 PJ-320D, U1 XIAO ESP32-C5

Commit message: REV C: D1 on the R7 row, symmetric rear jumpers
- D1 holes moved to y = 123 mm, the same row as R7's holes
- SJ2 (BIT 7) moved to the R5 row, mirroring SJ3 (BIT 8) on the R3 row
  around the middle of the resistor bank; labels on the outside; BIT 7
  traces rerouted
- Gerbers, drills, ZIPs, PDF, SVGs, STEP/GLB, renders and DRC/ERC
  regenerated (KiCad 10.0.7: DRC 0 / unconnected 0 / parity 0, ERC 0)
- REV C README updated

Co-Authored-By: Claude Opus 5.5 <noreply@anthropic.com>
Claude-Session: https://claude.ai/code/session_017AWz9uZd39iY6CDkhsBZb6
Parts:
- moved SJ2 4.65 mm to (122.0, 108.0)
- moved D1 0.70 mm to (115.7, 123.0)
Routing:
- net /DAC_EXT7: track 9.68 -> 14.7 mm
- net /DAC_EXT7_SW: track 5.62 -> 7.32 mm
- net /5V_XIAO: track 35.6 -> 34.9 mm
- net /5V_BAY: track 21.7 -> 22.4 mm
Changed lines of the file:
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@@
 	(footprint "C5VRX:D_DO-41_P7.62mm_Horizontal_Compact"
 		(layer "F.Cu")
-		(at 115.71 123.7)
+		(at 115.71 123)
 		(descr "DO-41 axial diode, 7.62 mm lead pitch, 1.7 mm pads / 1.0 mm drill for a tighter courtyard (C5VRX DIY REV C)")
 		(tags "Diode DO-41_SOD81 series Axial Horizontal pin pitch 7.62mm  length 5.2mm diameter 2.7mm")
@@
 	(footprint "Jumper:SolderJumper-2_P1.3mm_Open_Pad1.0x1.5mm"
 		(layer "B.Cu")
-		(at 120 103.8)
+		(at 122 108)
 		(descr "SMD Solder Jumper, 1x1.5mm Pads, 0.3mm gap, open")
 		(tags "solder jumper open")
@@
 	)
 	(gr_text "SJ2 BIT 7"
-		(at 120 105.7 0)
+		(at 122 106.3 0)
 		(layer "B.SilkS")
 		(effects
@@
 	)
 	(gr_text "SJ3 BIT 8"
-		(at 122 118.3 0)
+		(at 122 121.7 0)
 		(layer "B.SilkS")
 		(effects
@@
 	)
 	(segment
-		(start 120.65 103.8)
-		(end 123.72 103.8)
+		(start 122.65 104.5)
+		(end 124.15 103)
 		(width 0.25)
 		(layer "B.Cu")
@@
 	)
 	(segment
-		(start 123.72 103.8)
+		(start 122.65 108)
+		(end 122.65 104.5)
+		(width 0.25)
+		(layer "B.Cu")
+		(net "/DAC_EXT7_SW")
+	)
+	(segment
+		(start 124.15 103)
 		(end 125.52 102)
 		(width 0.25)
@@
 	)
 	(segment
+		(start 119.35 103.8)
+		(end 121.35 105.8)
+		(width 0.25)
+		(layer "B.Cu")
+		(net "/DAC_EXT7")
+	)
+	(segment
 		(start 111.5 103)
 		(end 112.3 103.8)
@@
 		(start 112.3 103.8)
 		(end 119.35 103.8)
+		(width 0.25)
+		(layer "B.Cu")
+		(net "/DAC_EXT7")
+	)
+	(segment
+		(start 121.35 105.8)
+		(end 121.35 108)
 		(width 0.25)
 		(layer "B.Cu")
@@
 	(segment
 		(start 115.71 119)
-		(end 115.71 123.7)
+		(end 115.71 123)
 		(width 0.5)
 		(layer "B.Cu")
@@
 	)
 	(segment
-		(start 123.33 123.7)
+		(start 123.33 123)
 		(end 123.33 126.9)
 		(width 0.5)
